File: _autosave-StartUP Board.kicad_sch (KiCad schematic)
At the start: 20 parts, among them J1 Conn_01x03_Socket, U2 TVS0500DRV, U3 ANT13SECQE

Commit message: Revised start up board, hopefully done
Parts:
- removed J1: Conn_01x03_Socket, Connector_Molex:Molex_Micro-Fit_3.0_43650-0300_1x03_P3.00mm_Horizontal, symbol Connector:Conn_01x03_Socket
- removed R10, R8, R9: 30k, Resistor_SMD:R_0402_1005Metric, symbol Device:R
- removed R5, R6, R7: 10k, Resistor_SMD:R_0402_1005Metric, symbol Device:R
- removed U2: TVS0500DRV, Package_SON:WSON-6-1EP_2x2mm_P0.65mm_EP1x1.6mm, symbol Power_Protection:TVS0500DRV
- added C5: 4.7 uF, Capacitor_SMD:C_0805_2012Metric, symbol Device:C
- added C6: 1 uF, Capacitor_SMD:C_0805_2012Metric, symbol Device:C
- added J2: Conn_01x04_Socket, Connector_Molex:Molex_Micro-Fit_3.0_43650-0400_1x04_P3.00mm_Horizontal, symbol Connector:Conn_01x04_Socket
- added Q1: NMOS, NX7002AK_215:SOT95P230X110-3N, symbol Simulation_SPICE:NMOS
- added TP1, TP2, TP3, TP4, TP5: TestPoint, TestPoint:TestPoint_Pad_D1.5mm, symbol Connector:TestPoint
- added U1: SN74LVC1G332DCKR, SN74LVC1G332DCKR:SOT65P210X110-6N, symbol SN74LVC1G332DCKR:SN74LVC1G332DCKR
- added VR1: TS9011SCX_RFG, TS9011SCX_RFG:VREG_TS9011SCX_RFG, symbol TS9011SCX_RFG:TS9011SCX_RFG
- AUX_12V1: footprint Connector_Molex:Molex_Micro-Fit_3.0_43650-0215_1x02_P3.00mm_Vertical -> Connector_Molex:Molex_Mega-Fit_76825-0002_2x01_P5.70mm_Horizontal; product number (none) -> WM1917-ND
- C1, C2, C3, C4: footprint Capacitor_SMD:C_0402_1005Metric -> Capacitor_SMD:C_0805_2012Metric; product number (none) -> 1276-1003-1-ND
- KEYSW_EXT1: product number (none) -> WM1863-ND
- R1, R2, R3, R4: footprint Resistor_SMD:R_0402_1005Metric -> Resistor_SMD:R_0805_2012Metric; product number (none) -> P100KADCT-ND
- U3: product number (none) -> 2449-ANT13SECQE-ND
Connections:
- net +12V: now also C5.1, Q1.1 (D), VR1.3 (VIN); no longer KEYSW_EXT1.5 (Pin_5)
- net GND: now also C5.2, C6.2, U1.2 (GND), VR1.1 (GND)
- net KEYSW_AUX: now also J2.2 (Pin_2), TP2.1, U1.1
- net KEYSW_CHARGE: now also J2.4 (Pin_4), TP4.1, U1.6
- net KEYSW_MAIN: now also J2.3 (Pin_3), TP3.1, U1.3
- new net: J2.1 (Pin_1), Q1.3 (S), TP5.1
- new net: Q1.2 (G), TP1.1, U1.4
- new net +3.3V: C6.1, KEYSW_EXT1.5 (Pin_5), U1.5 (VCC), VR1.2 (VOUT)
Other:
- moved on the sheet: KEYSW_EXT1
