File: StartUP Board.kicad_pcb (KiCad board)
At the start: 2 copper layers, 85.8 x 175 mm, 24 parts, among them J1 KEYSW_OUT, U2 D1, U3 ANT13SECQE

Commit message: finished
Parts:
- moved U3 63.5 mm to (185.0, 34.8)
- moved REF** 5.00 mm to (125.0, 60.2)
- moved REF** 4.76 mm to (203.5, 60.0)
Routing:
- net GND: track 105.7 -> 24.3 mm, vias 9 -> 8
- net /FNR_FWD: track 91.3 -> 55.7 mm
- net /FNR_REV: track 86.8 -> 53.2 mm
Other:
- outline, holes or cut-outs redrawn
- board text added: "Artemis 2026 Start-Up Board lrassett@purdue.edu"
- board text added: "C2"
- board text added: "F"
- board text added: "N"
- board text added: "R"
- board text added: "R1"
- board text removed: "8.7.A.3 switch labels at least 10mm tall - should switch just be seperate? is board too big (too expensive?)"
- board text removed: "<-- E-Stop mounting holes"
- board text removed: "FNR"
Changed lines of the file:
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@@
 		)
 		(property "Value" "R2"
-			(at 0.506709 1 90)
+			(at 0.49 -1 90)
 			(layer "F.SilkS")
 			(effects
@@
 		)
 		(property "Value" "R3"
-			(at 0.49 1 90)
+			(at 0.49 -1 90)
 			(layer "F.SilkS")
 			(effects
@@
 		)
 		(property "Value" "C4"
-			(at -0.246709 1 90)
+			(at 1.02 -1 90)
 			(layer "F.SilkS")
 			(effects
@@
 	(footprint "ANT13SECQE:ANT13SEC_CRS"
 		(layer "F.Cu")
-		(at 158 -22.674 90)
+		(at 185 34.826 90)
 		(tags "ANT13SECQE ")
 		(property "Reference" "U3"
@@
 		)
 		(property "Value" "C3"
-			(at -0.246709 1 90)
+			(at 1.02 -1 90)
 			(layer "F.SilkS")
 			(effects
@@
 		)
 		(property "Value" "R5"
-			(at -0.28 1 90)
+			(at 0.503291 1 90)
 			(layer "F.SilkS")
 			(effects
@@
 	(footprint "MountingHole:MountingHole_3.2mm_M3"
 		(layer "F.Cu")
-		(at 125 55.25)
+		(at 125 60.25)
 		(descr "Mounting Hole 3.2mm, M3, no annular, generated by kicad-footprint-generator mountinghole.py")
 		(tags "mountinghole M3")
@@
 		)
 		(property "Value" "R4"
-			(at 0.49 1 90)
+			(at 0.49 -1 90)
 			(layer "F.SilkS")
 			(effects
@@
 		)
 		(property "Value" "C1"
-			(at 0.503291 1.03 90)
+			(at 1.02 -0.97 90)
 			(layer "F.SilkS")
 			(effects
@@
 	(footprint "MountingHole:MountingHole_3.2mm_M3"
 		(layer "F.Cu")
-		(at 203.75 55.25)
+		(at 203.5 60)
 		(descr "Mounting Hole 3.2mm, M3, no annular, generated by kicad-footprint-generator mountinghole.py")
 		(tags "mountinghole M3")
@@
 	)
 	(gr_circle
-		(center 164.25 -76)
-		(end 194.4125 -76)
+		(center 164.5 -78.5)
+		(end 194.6625 -78.5)
 		(stroke
 			(width 0.1)
@@
 	)
 	(gr_arc
-		(start 156.242946 14.177778)
-		(mid 164.370232 9.75)
-		(end 172.5 14.173218)
+		(start 155.992946 -15.322222)
+		(mid 164.120232 -19.75)
+		(end 172.25 -15.326782)
 		(stroke
 			(width 0.05)
@@
 	)
 	(gr_line
-		(start 156.242946 14.17778)
-		(end 156.239953 24.673135)
+		(start 155.992946 -15.32222)
+		(end 155.989953 -4.826865)
 		(stroke
 			(width 0.05)
@@
 	)
 	(gr_line
-		(start 172.5 14.17322)
-		(end 172.5 24.682336)
+		(start 172.25 -15.32678)
+		(end 172.25 -4.817664)
 		(stroke
 			(width 0.05)
@@
 	)
 	(gr_circle
-		(center 149.25 -76)
-		(end 151.75 -76)
+		(center 149.5 -78.5)
+		(end 152 -78.5)
 		(stroke
 			(width 0.05)
@@
 	)
 	(gr_circle
-		(center 164.25 -76)
-		(end 176.25 -76)
+		(center 164.5 -78.5)
+		(end 176.5 -78.5)
 		(stroke
 			(width 0.05)
@@
 	)
 	(gr_circle
-		(center 179.25 -76)
-		(end 181.75 -76)
+		(center 179.5 -78.5)
+		(end 182 -78.5)
 		(stroke
 			(width 0.05)
@@
 	)
 	(gr_arc
-		(start 172.499998 24.682337)
-		(mid 164.367471 29.105553)
-		(end 156.239953 24.673138)
+		(start 172.249998 -4.817663)
+		(mid 164.117471 -0.394447)
+		(end 155.989953 -4.826862)
 		(stroke
 			(width 0.05)
@@
 		(layer "Edge.Cuts")
 	)
+	(gr_text "R1"
+		(at 137.5 41 90)
+		(layer "F.SilkS")
+		(effects
+			(font
+				(size 0.5 0.5)
+				(thickness 0.125)
+			)
+		)
+	)
 	(gr_text "OFF"
-		(at 123 25.5 0)
+		(at 122.75 -4 0)
 		(layer "F.SilkS")
 		(effects
@@
 	)
 	(gr_text "POWER"
-		(at 138 5.5 0)
+		(at 137.75 -24 0)
 		(layer "F.SilkS")
 		(effects
@@
 		)
 	)
+	(gr_text "C2"
+		(at 142 46 90)
+		(layer "F.SilkS")
+		(effects
+			(font
+				(size 0.5 0.5)
+				(thickness 0.125)
+			)
+		)
+	)
 	(gr_text "ON"
-		(at 179.5 25.5 0)
+		(at 179.25 -4 0)
 		(layer "F.SilkS")
 		(effects
@@
 	)
 	(gr_text "CHG\n"
-		(at 149.25 46.5 0)
+		(at 149 17 0)
 		(layer "F.SilkS")
 		(effects
@@
 		)
 	)
-	(gr_text "FNR"
-		(at 165.75 -42.5 270)
+	(gr_text "F"
+		(at 189.5 24.5 0)
 		(layer "F.SilkS")
 		(effects
 			(font
-				(size 10 10)
+				(size 8 10)
 				(thickness 1.25)
 			)
@@
 		)
 	)
-	(gr_text "8.7.A.3 switch labels at least 10mm tall \n- should switch just be seperate?\n\nis board too big (too expensive?)\n"
-		(at 258.75 18.5 0)
-		(layer "User.2")
+	(gr_text "R\n"
+		(at 188.25 46.75 0)
+		(layer "F.SilkS")
 		(effects
 			(font
-				(size 5 5)
-				(thickness 0.625)
+				(size 8 10)
+				(thickness 1.25)
 			)
 			(justify left bottom)
 		)
 	)
-	(gr_text "<-- E-Stop mounting holes"
-		(at 261.75 -83.5 0)
-		(layer "User.2")
+	(gr_text "Artemis 2026\nStart-Up Board\nlrassett@purdue.edu"
+		(at 132.25 54 90)
+		(layer "F.SilkS")
+		(effects
+			(font
+				(size 2 2)
+				(thickness 0.125)
+			)
+			(justify left bottom)
+		)
+	)
+	(gr_text "N"
+		(at 188.5 35.25 0)
+		(layer "F.SilkS")
 		(effects
 			(font
-				(size 5 5)
-				(thickness 0.625)
+				(size 8 10)
+				(thickness 1.25)
 			)
 			(justify left bottom)
@@
 	)
 	(segment
-		(start 159.6321 -24.3061)
-		(end 159.6321 -33.002038)
-		(width 0.5)
-		(layer "F.Cu")
-		(net 1)
-	)
-	(segment
 		(start 141.326709 32.673291)
 		(end 141.273291 32.673291)
@@
 	)
 	(segment
-		(start 158 -22.674)
-		(end 159.6321 -24.3061)
-		(width 0.5)
-		(layer "F.Cu")
-		(net 1)
-	)
-	(segment
-		(start 157.323962 -33.9581)
-		(end 152 -28.634138)
-		(width 0.5)
-		(layer "F.Cu")
-		(net 1)
-	)
-	(segment
 		(start 143.25 43.486581)
 		(end 143.25 43)
@@
 	)
 	(segment
-		(start 152 -28.634138)
-		(end 152 31.5)
-		(width 0.5)
-		(layer "F.Cu")
-		(net 1)
-	)
-	(segment
 		(start 148.773291 33.283291)
 		(end 148.773291 33.933291)
@@
 	)
 	(segment
-		(start 159.6321 -33.002038)
-		(end 158.676038 -33.9581)
-		(width 0.5)
-		(layer "F.Cu")
-		(net 1)
-	)
-	(segment
 		(start 140.75 43.676958)
 		(end 140.75 43)
@@
 	)
 	(segment
-		(start 158.676038 -33.9581)
-		(end 157.323962 -33.9581)
-		(width 0.5)
-		(layer "F.Cu")
-		(net 1)
-	)
-	(segment
 		(start 146 42.75)
 		(end 145.75 43)
@@
 		(net 1)
 	)
-	(via
-		(at 152 31.5)
-		(size 0.5)
-		(drill 0.3)
-		(layers "F.Cu" "B.Cu")
-		(net 1)
-	)
 	(segment
 		(start 147.0759 60.25)
@@
 	)
 	(segment
-		(start 149.5 36.25)
-		(end 153 32.75)
-		(width 0.5)
-		(layer "F.Cu")
-		(net 7)
-	)
-	(segment
-		(start 153 32.75)
-		(end 153 -27.326)
+		(start 185 25.174)
+		(end 167.924 42.25)
 		(width 0.5)
 		(layer "F.Cu")
@@
 	)
 	(segment
-		(start 153 -27.326)
-		(end 158 -32.326)
-		(width 0.5)
-		(layer "F.Cu")
-		(net 7)
-	)
-	(segment
-		(start 149.5 42.25)
-		(end 149.5 36.25)
+		(start 167.924 42.25)
+		(end 149.5 42.25)
 		(width 0.5)
 		(layer "F.Cu")
@@
 	)
 	(segment
-		(start 150.5 42.75)
-		(end 150.5 36.75)
-		(width 0.5)
-		(layer "F.Cu")
-		(net 8)
-	)
-	(segment
-		(start 158 -27.5)
-		(end 153.75 -23.25)
-		(width 0.5)
-		(layer "F.Cu")
-		(net 8)
-	)
-	(segment
-		(start 153.75 -23.25)
-		(end 153.75 33.5)
-		(width 0.5)
-		(layer "F.Cu")
-		(net 8)
-	)
-	(segment
-		(start 153.75 33.5)
-		(end 150.5 36.75)
+		(start 185 30)
+		(end 172 43)
 		(width 0.5)
 		(layer "F.Cu")
@@
 	)
 	(segment
-		(start 150.25 43)
-		(end 150.5 42.75)
+		(start 172 43)
+		(end 150.25 43)
 		(width 0.5)
 		(layer "F.Cu")

Commit message: revised start up board 3-7-26
Other:
- board text added: "TOP - GND"
Changed lines of the file:
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@@
+		)
+	)
+	(gr_text "TOP - GND"
+		(at 136.25 62.5 90)
+		(layer "F.SilkS")
+		(effects
+			(font
+				(size 1 1)
+				(thickness 0.1)
+			)
+			(justify left bottom)
 		)
 	)

Commit message: Revised start up board, hopefully done
Parts:
- removed GPIO6: FNR_OUT, Connector_Molex:Molex_Micro-Fit_3.0_43650-0200_1x02_P3.00mm_Horizontal
- removed J1: KEYSW_OUT, Connector_Molex:Molex_Micro-Fit_3.0_43650-0300_1x03_P3.00mm_Horizontal
- removed R10: R10, Resistor_SMD:R_0402_1005Metric
- removed R5: R5, Resistor_SMD:R_0402_1005Metric
- removed R6: R6, Resistor_SMD:R_0402_1005Metric
- removed R7: R7, Resistor_SMD:R_0402_1005Metric
- removed R8: R8, Resistor_SMD:R_0402_1005Metric
- removed R9: R9, Resistor_SMD:R_0402_1005Metric
- removed the REF** at (125.0, -107.8)
- removed the REF** at (203.8, -107.8)
- removed U2: D1, Package_SON:WSON-6-1EP_2x2mm_P0.65mm_EP1x1.6mm
- added C5: 4.7 uF, Capacitor_SMD:C_0805_2012Metric, F.Cu at (152.8, 44.2)
- added C6: 1 uF, Capacitor_SMD:C_0805_2012Metric, F.Cu at (155.8, 41.2)
- added FNR: GPIO7, Connector_Molex:Molex_Micro-Fit_3.0_43650-0200_1x02_P3.00mm_Horizontal, F.Cu at (174.8, 52.8)
- added OUTPUT: Conn_01x04_Socket, Connector_Molex:Molex_Micro-Fit_3.0_43650-0400_1x04_P3.00mm_Horizontal, F.Cu at (153.2, 52.9)
- added Q1: NMOS, NX7002AK_215:SOT95P230X110-3N, F.Cu at (155.1, 48.8)
- added TP1: TestPoint, TestPoint:TestPoint_Pad_D1.5mm, B.Cu at (147.2, 45.0)
- added TP2: TestPoint, TestPoint:TestPoint_Pad_D1.5mm, B.Cu at (144.2, 46.8)
- added TP3: TestPoint, TestPoint:TestPoint_Pad_D1.5mm, B.Cu at (147.0, 50.0)
- added TP4: TestPoint, TestPoint:TestPoint_Pad_D1.5mm, F.Cu at (138.9, 49.2)
- added TP5: TestPoint, TestPoint:TestPoint_Pad_D1.5mm, B.Cu at (151.8, 49.8)
- added U1: SN74LVC1G332DCKR, SN74LVC1G332DCKR:SOT65P210X110-6N, F.Cu at (149.8, 49.0)
- added VR1: TS9011SCX_RFG, TS9011SCX_RFG:VREG_TS9011SCX_RFG, F.Cu at (155.7, 44.2)
- AUX_12V1: footprint Micro-Fit 3.0 Right-Angle Header:CONN_SD-43045-001_02_MOL -> Connector_Molex:Molex_Mega-Fit_76825-0002_2x01_P5.70mm_Horizontal
- C1: value C1 -> 0.1u; footprint Capacitor_SMD:C_0402_1005Metric -> Capacitor_SMD:C_0805_2012Metric
- C2: footprint Capacitor_SMD:C_0402_1005Metric -> Capacitor_SMD:C_0805_2012Metric
- C3: value C3 -> 0.1u; footprint Capacitor_SMD:C_0402_1005Metric -> Capacitor_SMD:C_0805_2012Metric
- C4: value C4 -> 0.1u; footprint Capacitor_SMD:C_0402_1005Metric -> Capacitor_SMD:C_0805_2012Metric
- KEYSW_EXT1: value KEYSW_EXT -> Conn_01x05_Socket; moved to B.Cu
- R1: footprint Resistor_SMD:R_0402_1005Metric -> Resistor_SMD:R_0805_2012Metric
- R2: value R2 -> 100k; footprint Resistor_SMD:R_0402_1005Metric -> Resistor_SMD:R_0805_2012Metric
- R3: value R3 -> 100k; footprint Resistor_SMD:R_0402_1005Metric -> Resistor_SMD:R_0805_2012Metric
- R4: value R4 -> 100k; footprint Resistor_SMD:R_0402_1005Metric -> Resistor_SMD:R_0805_2012Metric
- moved R4 53.7 mm to (199.2, 48.4)
- moved C4 53.3 mm to (199.2, 44.2), turned to 90 degrees
- moved R3 53.2 mm to (196.2, 48.4)
- moved R2 53.0 mm to (193.5, 48.4)
- moved C3 52.8 mm to (196.2, 44.2), turned to 90 degrees
- moved R1 52.7 mm to (190.8, 48.4)
- moved C2 52.5 mm to (193.5, 44.2), turned to 90 degrees
- moved C1 52.2 mm to (190.8, 44.2), turned to 90 degrees
- moved AUX_12V1 23.2 mm to (162.5, 46.0), turned to 180 degrees
- moved U3 13.7 mm to (196.0, 26.7)
- moved KEYSW_EXT1 10.0 mm to (195.2, 60.8)
Connections:
- KEYSW_EXT1 pad 5: +12V -> +3.3V
Routing:
- net Net-(J1-Pin_1): track 135.9 -> 0.00 mm, vias 6 -> 0
- net +3.3V: track 0.00 -> 65.5 mm, vias 0 -> 1
- net +12V: track 41.4 -> 0.00 mm
- net /KEYSW_OFF: track 52.6 -> 19.9 mm
- net /KEYSW_CHARGE: track 57.3 -> 79.0 mm
- net /KEYSW_MAIN: track 56.2 -> 77.1 mm
- net /KEYSW_AUX: track 57.2 -> 76.7 mm
- net GND: track 24.3 -> 5.58 mm, vias 8 -> 3
- net /FNR_REV: track 53.2 -> 39.8 mm, vias 1 -> 0
- net Net-(Q1-G): track 0.00 -> 9.92 mm, vias 0 -> 1
- net /FNR_FWD: track 55.7 -> 45.8 mm, vias 2 -> 0
- net Net-(J2-Pin_1): track 0.00 -> 7.70 mm
- added copper zone on F.Cu, net +12V
- added copper zone on F.Cu, net GND
Other:
- board size 85.8 x 175 mm -> 85.8 x 55 mm
- board text added: "Mmmmm"
- board text removed: "Artemis 2026 Start-Up Board lrassett@purdue.edu"
- board text removed: "C2"
- board text removed: "CHG"
- board text removed: "F"
- board text removed: "N"
- board text removed: "OFF"
- board text removed: "ON"
- board text removed: "POWER"
- board text removed: "R"
- board text removed: "R1"
- board text removed: "TOP - GND"

Commit message: Man added
Parts:
- added G***: LOGO, LOGO, F.Cu at (133.4, 16.6)
Other:
- board text added: "Artemis 2026 Start up Board yang2575@purdue.edu"
- board text removed: "Mmmmm"

Commit message: upload vivian iteration of PCB
Parts:
- removed AUX_12V1: GND, Connector_Molex:Molex_Mega-Fit_76825-0002_2x01_P5.70mm_Horizontal
- removed FNR: GPIO7, Connector_Molex:Molex_Micro-Fit_3.0_43650-0200_1x02_P3.00mm_Horizontal
- removed G***: LOGO, LOGO
- removed KEYSW_EXT1: Conn_01x05_Socket, Connector_Molex:Molex_Micro-Fit_3.0_43650-0500_1x05_P3.00mm_Horizontal
- removed OUTPUT: Conn_01x04_Socket, Connector_Molex:Molex_Micro-Fit_3.0_43650-0400_1x04_P3.00mm_Horizontal
- removed Q1: NMOS, NX7002AK_215:SOT95P230X110-3N
- removed REF**: H3, MountingHole:MountingHole_3.2mm_M3
- removed REF**: H4, MountingHole:MountingHole_3.2mm_M3
- removed TP1, TP2, TP3, TP4, TP5: TestPoint, TestPoint:TestPoint_Pad_D1.5mm
- removed U3: ANT13SECQE, ANT13SECQE:ANT13SEC_CRS
- removed VR1: TS9011SCX_RFG, TS9011SCX_RFG:VREG_TS9011SCX_RFG
- added H1: MountingHole, MountingHole:MountingHole_3.2mm_M3, F.Cu at (125.0, 60.2)
- added H2: MountingHole, MountingHole:MountingHole_3.2mm_M3, F.Cu at (203.8, 60.2)
- added IC1: AP7380-33W5-7, AP7380-33W5-7:AP7380-33W5-7, F.Cu at (150.8, 45.7)
- added J1: Conn_01x05_Socket, Connector_Molex:Molex_Micro-Fit_3.0_43650-0500_1x05_P3.00mm_Horizontal, B.Cu at (184.0, 59.7)
- added J2: ~, Connector_Molex:Molex_Micro-Fit_3.0_43650-0200_1x02_P3.00mm_Horizontal, F.Cu at (141.1, 53.8)
- added J3: ~, Connector_Molex:Molex_Micro-Fit_3.0_43650-0200_1x02_P3.00mm_Horizontal, F.Cu at (193.5, 53.9)
- added J4: ~, Connector_Molex:Molex_Mega-Fit_76825-0002_2x01_P5.70mm_Horizontal, F.Cu at (162.2, 47.0)
- added J5: ~, Connector_Molex:Molex_Micro-Fit_3.0_43650-0200_1x02_P3.00mm_Horizontal, F.Cu at (152.6, 53.8)
- added R5: 100k, Resistor_SMD:R_0805_2012Metric, F.Cu at (135.3, 49.9)
- added R6: 100k, Resistor_SMD:R_0805_2012Metric, F.Cu at (132.3, 49.9)
- added U2: CD4049UBDR, CD4049UBDR:D16-M, F.Cu at (142.2, 45.7)
- C5: value 4.7 uF -> 1 uF
- U1: value SN74LVC1G332DCKR -> ANT13SECQE; footprint SN74LVC1G332DCKR:SOT65P210X110-6N -> ANT13SEC_CRS:ANT13SEC_CRS
- moved U1 48.9 mm to (194.6, 29.1)
- moved C1 16.6 mm to (174.2, 45.0), turned to 0 degrees
- moved R1 16.6 mm to (174.2, 47.8), turned to 180 degrees
- moved R2 15.5 mm to (178.0, 47.8), turned to 180 degrees
- moved C2 15.5 mm to (178.1, 44.9), turned to 0 degrees
- moved R3 14.4 mm to (181.9, 47.8), turned to 180 degrees
- moved C3 14.3 mm to (181.9, 44.7), turned to 0 degrees
- moved R4 13.6 mm to (185.7, 47.8), turned to 180 degrees
- moved C4 13.6 mm to (185.7, 44.7), turned to 0 degrees
- moved C6 9.23 mm to (150.8, 49.0), turned to 180 degrees
- moved C5 2.63 mm to (150.8, 42.4), turned to 180 degrees
Connections:
- C5 pad 1: +12V -> /KEYSW_CHARGE
- U1 pad 1: /KEYSW_AUX -> /FNR_REV
- U1 pad 3: /KEYSW_MAIN -> /FNR_FWD
Routing:
- net /KEYSW_MAIN: track 77.1 -> 15.2 mm
- net /KEYSW_AUX: track 76.7 -> 16.0 mm
- net +3.3V: track 65.5 -> 7.18 mm, vias 1 -> 0
- net +12V: track 0.00 -> 56.7 mm, vias 0 -> 1
- net /KEYSW_OFF: track 19.9 -> 67.5 mm
- net /KEYSW_CHARGE: track 79.0 -> 57.8 mm
- net /FNR_REV: track 39.8 -> 25.3 mm
- net /KeySwitch_LV: track 0.00 -> 12.2 mm
- net Net-(Q1-G): track 9.92 -> 0.00 mm, vias 1 -> 0
- net /FNR_FWD: track 45.8 -> 36.2 mm
- net GND: track 5.58 -> 14.3 mm, vias 3 -> 108
- net Net-(J2-Pin_1): track 7.70 -> 0.00 mm
- removed copper zone on F.Cu, net +12V
Other:
- board text added: "*"
- board text added: "Artemis 2026 Start Up Board v2 yang2575@purdue.edu lrassett@purdue.edu siskb@purdue.edu vrschmal@gmail.com"
- board text removed: "Artemis 2026 Start up Board yang2575@purdue.edu"
