File: StartUP Board.kicad_sch (KiCad schematic)
At the start: 22 parts, among them J1 Conn_01x03_Socket, U1 TVS0500DRV, U2 TVS0500DRV, U3 ANT13SECQE, U4 TVS0500DRV

Commit message: revised start up board 3-7-26
Parts:
- removed J1: Conn_01x03_Socket, Connector_Molex:Molex_Micro-Fit_3.0_43650-0300_1x03_P3.00mm_Horizontal, symbol Connector:Conn_01x03_Socket
- removed R10, R8, R9: 30k, Resistor_SMD:R_0402_1005Metric, symbol Device:R
- removed R5, R6, R7: 10k, Resistor_SMD:R_0402_1005Metric, symbol Device:R
- removed U1, U2, U4: TVS0500DRV, Package_SON:WSON-6-1EP_2x2mm_P0.65mm_EP1x1.6mm, symbol Power_Protection:TVS0500DRV
- added C5: 4.7 uF, Capacitor_SMD:C_0805_2012Metric, symbol Device:C
- added C6: 1 uF, Capacitor_SMD:C_0805_2012Metric, symbol Device:C
- added J2: Conn_01x04_Socket, Connector_Molex:Molex_Micro-Fit_3.0_43650-0400_1x04_P3.00mm_Horizontal, symbol Connector:Conn_01x04_Socket
- added Q1: NMOS, NX7002AK_215:SOT95P230X110-3N, symbol Simulation_SPICE:NMOS
- added TP1, TP2, TP3, TP4, TP5: TestPoint, TestPoint:TestPoint_Pad_1.5x1.5mm, symbol Connector:TestPoint
- added U1: SN74LVC1G332DCKR, SN74LVC1G332DCKR:SOT65P210X110-6N, symbol SN74LVC1G332DCKR:SN74LVC1G332DCKR
- added VR1: TS9011SCX_RFG, TS9011SCX_RFG:VREG_TS9011SCX_RFG, symbol TS9011SCX_RFG:TS9011SCX_RFG
- AUX_12V1: product number (none) -> WM1917-ND
- C1, C2, C3, C4: footprint Capacitor_SMD:C_0402_1005Metric -> Capacitor_SMD:C_0805_2012Metric; product number (none) -> 1276-1003-1-ND
- KEYSW_EXT1: product number (none) -> WM1863-ND
- R1, R2, R3, R4: footprint Resistor_SMD:R_0402_1005Metric -> Resistor_SMD:R_0805_2012Metric; product number (none) -> P100KADCT-ND
- U3: footprint ANT13SECQE:ANT13SEC_CRS -> Capacitor_SMD:C_0805_2012Metric; product number (none) -> 2449-ANT13SECQE-ND
Connections:
- net +12V: now also C5.1, Q1.1 (D), VR1.3 (VIN); no longer KEYSW_EXT1.5 (Pin_5)
- net GND: now also C5.2, C6.2, U1.2 (GND), VR1.1 (GND)
- net KEYSW_AUX: now also J2.2 (Pin_2), TP2.1, U1.1
- net KEYSW_CHARGE: now also J2.4 (Pin_4), TP4.1, U1.6
- net KEYSW_MAIN: now also J2.3 (Pin_3), TP3.1, U1.3
- new net: J2.1 (Pin_1), Q1.3 (S), TP5.1
- new net: Q1.2 (G), TP1.1, U1.4
- new net +3.3V: C6.1, KEYSW_EXT1.5 (Pin_5), U1.5 (VCC), VR1.2 (VOUT)
Other:
- moved on the sheet: KEYSW_EXT1

Commit message: Revised start up board, hopefully done
Parts:
- U3: footprint Capacitor_SMD:C_0805_2012Metric -> ANT13SECQE:ANT13SEC_CRS
Changed lines of the file:
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@@
 			)
 		)
-		(property "Footprint" "Capacitor_SMD:C_0805_2012Metric"
+		(property "Footprint" "ANT13SECQE:ANT13SEC_CRS"
 			(at 73.66 57.15 0)
 			(effects

Commit message: Man added
Parts:
- AUX_12V1: footprint Connector_Molex:Molex_Micro-Fit_3.0_43650-0215_1x02_P3.00mm_Vertical -> Connector_Molex:Molex_Mega-Fit_76825-0002_2x01_P5.70mm_Horizontal
- TP1, TP2, TP3, TP4, TP5: footprint TestPoint:TestPoint_Pad_1.5x1.5mm -> TestPoint:TestPoint_Pad_D1.5mm
Other:
- note added: "2"
Changed lines of the file:
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@@
 		)
 	)
+	(text "2"
+		(exclude_from_sim no)
+		(at 270.002 193.294 0)
+		(effects
+			(font
+				(size 1.27 1.27)
+			)
+		)
+	)
 	(text "FNR Switch"
 		(exclude_from_sim no)
@@
 			)
 		)
-		(property "Footprint" "TestPoint:TestPoint_Pad_1.5x1.5mm"
+		(property "Footprint" "TestPoint:TestPoint_Pad_D1.5mm"
 			(at 119.38 116.84 0)
 			(effects
@@
 			)
 		)
-		(property "Footprint" "TestPoint:TestPoint_Pad_1.5x1.5mm"
+		(property "Footprint" "TestPoint:TestPoint_Pad_D1.5mm"
 			(at 101.6 121.92 0)
 			(effects
@@
 			)
 		)
-		(property "Footprint" "TestPoint:TestPoint_Pad_1.5x1.5mm"
+		(property "Footprint" "TestPoint:TestPoint_Pad_D1.5mm"
 			(at 104.14 124.46 0)
 			(effects
@@
 			)
 		)
-		(property "Footprint" "TestPoint:TestPoint_Pad_1.5x1.5mm"
+		(property "Footprint" "TestPoint:TestPoint_Pad_D1.5mm"
 			(at 100.33 100.33 0)
 			(effects
@@
 			)
 		)
-		(property "Footprint" "TestPoint:TestPoint_Pad_1.5x1.5mm"
+		(property "Footprint" "TestPoint:TestPoint_Pad_D1.5mm"
 			(at 99.06 119.38 0)
 			(effects
@@
 			)
 		)
-		(property "Footprint" "Connector_Molex:Molex_Micro-Fit_3.0_43650-0215_1x02_P3.00mm_Vertical"
+		(property "Footprint" "Connector_Molex:Molex_Mega-Fit_76825-0002_2x01_P5.70mm_Horizontal"
 			(at 152.4 100.33 0)
 			(effects

Commit message: upload vivian iteration of PCB
Parts:
- removed J2: Conn_01x04_Socket, Connector_Molex:Molex_Micro-Fit_3.0_43650-0400_1x04_P3.00mm_Horizontal, symbol Connector:Conn_01x04_Socket
- removed Q1: NMOS, NX7002AK_215:SOT95P230X110-3N, symbol Simulation_SPICE:NMOS
- removed TP1, TP2, TP3, TP4, TP5: TestPoint, TestPoint:TestPoint_Pad_D1.5mm, symbol Connector:TestPoint
- removed U1: SN74LVC1G332DCKR, SN74LVC1G332DCKR:SOT65P210X110-6N, symbol SN74LVC1G332DCKR:SN74LVC1G332DCKR
- removed U3: ANT13SECQE, ANT13SECQE:ANT13SEC_CRS, symbol ANT13SECQE:ANT13SECQE
- removed VR1: TS9011SCX_RFG, TS9011SCX_RFG:VREG_TS9011SCX_RFG, symbol TS9011SCX_RFG:TS9011SCX_RFG
- added H1, H2: MountingHole, MountingHole:MountingHole_3.2mm_M3, symbol Mechanical:MountingHole
- added IC1: AP7380-33W5-7, AP7380-33W5-7:AP7380-33W5-7, symbol AP7380-33W5-7:AP7380-33W5-7
- added J2, J5: ~, Connector_Molex:Molex_Micro-Fit_3.0_43650-0200_1x02_P3.00mm_Horizontal, symbol Connector:Conn_01x02_Socket
- added R5, R6: 100k, Resistor_SMD:R_0805_2012Metric, symbol Device:R
- added U1: ANT13SECQE, ANT13SEC_CRS:ANT13SEC_CRS, symbol 2026-03-24_19-36-38:ANT13SECQE
- added U2: CD4049UBDR, CD4049UBDR:D16-M, symbol CD4049UBDR:CD4049UBDR
- C5: value 4.7 uF -> 1 uF
- J3: renamed from GPIO6; value GPIO7 -> ~
- J4: renamed from AUX_12V1; value GND -> ~
- renumbered KEYSW_EXT1 to J1
Connections:
- net +12V: now also J1.5 (Pin_5), J2.1 (Pin_1), R5.1, U2.1 (VCC); no longer C5.1
- net +3.3V: now also IC1.5 (VOUT), J5.1 (Pin_1); no longer J1.5 (Pin_5)
- net FNR_FWD: now also U1.3
- net FNR_REV: now also U1.1
- net GND: now also IC1.2 (GND), J5.2 (Pin_2), R6.2, U1.2, U2.8 (VSS)
- net KEYSW_CHARGE: now also C5.1, IC1.1 (VIN), IC1.3 (EN)
- net KEYSW_OFF: now also U2.3 (A)
- new net KeySwitch_LV: J2.2 (Pin_2), R5.2, R6.1, U2.2 (G=*A)
Other:
- note added: "External Keyswitch Connector"
- note added: "FNR Switch & Signal Connector"
- note added: "Output Signals"
- note added: "Power"
- note removed: "FNR Switch"
- note removed: "external keyswitch connector"
- note removed: "gpio outputs to pico"
- note removed: "power from aux"
- moved on the sheet: C1, C2, C3, C4, C5, C6, J1, R1, R2, R3, R4
